File: ovrBeaconGateway-wifi.sch (KiCad schematic (older format))
At the start: 35 parts, among them J1 USB_MICROB_RA_LONG, J2 CONN_RJ45_RA, Q1 BJT_NPN_1.5A_25V, Q2 BJT_NPN_1.5A_25V, Q3 FET_NP_5A/3A_60V, U1 SILICONLABS_SI7050, U2 TOREX_XC6210, U3 FTDI_RT232RL, U4 ESP32-WROOM, U5 INTERSIL_ISL32602EFBZ

Commit message: Included an optional BLE121 on this module to allow for stand-alone long range operation
Parts:
- added C4: C_0.1uF_10v_0603, ovrEngineered:C_0603, symbol C_0.1uF_10v_0603
- added U6: BLUEGIGA_BLE121, ovrEngineered:BLE121, symbol BLUEGIGA_BLE121
Connections:
- net +3V3: now also C4.1, U6.13 (AVCC), U6.23 (DVCC)
- net BTLE_POWER_ENABLE: now also U6.7 (~RESET)
- net ESP32-CTS_BTLE-RTS: now also U6.10 (P0_5)
- net ESP32-RTS_BTLE-CTS: now also U6.9 (P0_4)
- net ESP32-RX_BTLE-TX: now also U6.8 (P0_3)
- net ESP32-TX_BTLE-RX: now also U6.4 (PO_2)
- net GND: now also C4.2, U6.1 (GND), U6.14 (GND), U6.15 (GND), U6.16 (GND), U6.2 (GND), U6.22 (GND), U6.3 (GND), U6.31 (GND), U6.32 (GND), U6.33 (GND), U6.34 (GND), U6.35 (GND), U6.36 (GND)
- no-connect marks 29 -> 44
Other:
- note added: "High-Power BTLE"
- note added: "Power Control to External BTLE"
- note added: "RS422 converter and RJ45 to External BTLE"
- note added: "WiFi Module\nLow-Power BTLE"
- note removed: "Power Control to BTLE"
- note removed: "RS422 converter and RJ45 to BTLE"
- note removed: "WiFi Module"
- moved on the sheet: Q3, R14, R15, U4

Commit message: Initial commit of second revision changes
Parts:
- removed D1: LED_GREEN_0603, ovrEngineered:D_0603, symbol LED_GREEN_0603
- removed D2: LED_RED_0603, ovrEngineered:D_0603, symbol LED_RED_0603
- removed D3: CREE_CLV1A_FKB, ovrEngineered:CREE_CLV1A_FKB, symbol CREE_CLV1A_FKB
- removed D4: LED_BLUE_0603, ovrEngineered:D_0603, symbol LED_BLUE_0603
- removed R1, R18: R_402_1%_0603, ovrEngineered:R_0603, symbol R_402_1%_0603
- removed R11: R_5.1K_1%_0603, ovrEngineered:R_0603, symbol R_5.1K_1%_0603
- removed R6, R7: R_10K_1%_0603, ovrEngineered:R_0603, symbol R_10K_1%_0603
- added D1, D2: CREE_CLV1A_FKB, ovrEngineered:CREE_CLV1A_FKB, symbol CREE_CLV1A_FKB
- added J3: CONN_DBG_PDI, ovrEngineered:TC2030-IDC, symbol CONN_DBG_PDI
- added J4: CONN_1.27MM_5X2, ovrEngineered:20021111-00010T4LF, symbol CONN_1.27MM_5X2
- added R1, R11: R_12K_1%_0603, ovrEngineered:R_0603, symbol R_12K_1%_0603
- added R18: R_10K_1%_0603, ovrEngineered:R_0603, symbol R_10K_1%_0603
- added R19, R20, R21, R22: R_0_0603, ovrEngineered:R_0603, symbol R_0_0603
- added R6, R7: R_402_1%_0603, ovrEngineered:R_0603, symbol R_402_1%_0603
- added SW1: ESWITCH_TL3315NF100Q, ovrEngineered:TL3315NF100Q, symbol ESWITCH_TL3315NF100Q
- added U7: LITEON_LTR-329ALS, ovrEngineered:LITEON_LTR-329ALS, symbol LITEON_LTR-329ALS
Connections:
- net +3V3: now also R13.1, U5.4 (DE), D1.2 (ANODE), D2.2 (ANODE), J3.2 (VCC), J4.1, R1.1, R11.1, U7.1 (VCC)
- net +5V: now also R14.2; no longer R14.1
- net BTLE_POWER_ENABLE: now also U4.26 (IO4), R18.2; no longer U4.24 (IO2/strap), U6.7 (~RESET)
- net ESP32-CTS_BTLE-RTS: now also U4.13 (IO14); no longer U4.36 (IO22)
- net ESP32-RTS_BTLE-CTS: now also U4.16 (IO13); no longer U4.33 (IO21)
- net ESP32-RX_BTLE-TX: now also U4.27 (IO16), U5.2 (RO); no longer U4.28 (IO17), U5.5 (DI)
- net ESP32-RX_DBG-TX: now also J3.3 (TX)
- net ESP32-TX_BTLE-RX: now also U4.28 (IO17), U5.5 (DI); no longer U4.27 (IO16), U5.2 (RO)
- net ESP32-TX_DBG-RX: now also J3.4 (RX)
- net ESP32_EN: now also J3.1 (PDI_DATA)
- net ESP32_IO0: now also J3.5 (PDI_CLK), R11.2
- net GND: now also U5.3 (~RE), J3.6 (GND), J4.2, R21.2, R22.2, SW1.3, SW1.4, U7.2 (GND); no longer R13.2
- net at R3.1: now also D1.4 (CATHOD_GREEN)
- net at R5.1: now also D2.1 (CATHODE_RED)
- net at R4.1: now also D1.3 (CATHODE_BLUE)
- net at R2.1: now also D1.1 (CATHODE_RED)
- net at Q3.4, Q3.7, Q3.8: now also R14.1; no longer R14.2
- net LED_WIFI_R: now reaches U4.11 (IO26)
- net LED_WIFI_R: now also R2.2
- net ~VAR_IHP: now reaches U4.30 (IO18)
- net ~VAR_IHP: now also R22.1
- net SDA_ESP32: now reaches U4.31 (IO19)
- net SDA_ESP32: now also R19.1
- net P2_1/PROG: now reaches U6.20 (P2_1)
- net P2_1/PROG: now also J4.3
- net P2_2/PROG: now reaches U6.21 (P2_2)
- net P2_2/PROG: now also J4.4
- net SCL_BLE121: now reaches U6.24 (SCL)
- net SCL_BLE121: now also R13.2, U1.6 (SCL), R20.2, U7.4 (SCL)
- net SDA_BLE121: now reaches U6.25 (SDA)
- net SDA_BLE121: now also R12.2, U1.1 (SDA), R19.2, U7.3 (SDA)
- net +5V_SWITCHED: no longer names the net of J2.1 (W/O), Q3.5, Q3.6
- removed net 422_DE: R13.1, U4.16 (IO13), U5.4 (DE)
- net LED_BTLE_ACT renamed SW_WIFI_PROV
- net SW_WIFI_PROV: now also R1.2, SW1.1, SW1.2
- removed net LED_ERROR: R2.2, U4.13 (IO14)
- net LED_RGB_B renamed LED_BTLE_R
- net LED_BTLE_R: now also U4.8 (IO32); no longer U4.10 (IO25)
- net LED_RGB_G renamed LED_WIFI_B
- net LED_WIFI_B: now also U4.10 (IO25); no longer U4.9 (IO33)
- net LED_RGB_R renamed LED_WIFI_G
- net LED_WIFI_G: now also U4.9 (IO33); no longer U4.8 (IO32)
- net SCL renamed LED_BTLE_B
- net LED_BTLE_B: now also R7.2; no longer U1.6 (SCL)
- net SDA renamed LED_BTLE_G
- net LED_BTLE_G: now also R6.2; no longer U1.1 (SDA)
- removed net ~422_RE: R12.2, U4.14 (IO12/strap), U5.3 (~RE)
- new net: D2.3 (CATHODE_BLUE), R7.1
- new net: D2.4 (CATHOD_GREEN), R6.1
- new net SCL_ESP32: R20.1, U4.33 (IO21)
- new net ~BLE121_RESET: J4.8, R18.1, U6.7 (~RESET)
- new net ~VAR_EXT: R21.1, U4.14 (IO12/strap)
- no-connect marks 44 -> 43
Other:
- note added: "+5V Switched Supply"
- note added: "BTLE Activity LED"
- note added: "BTLE Variant: External"
- note added: "BTLE Variant: Internal"
- note added: "BTLE Variant: Internal High-Power"
- note added: "BTLE Variant: \n Internal\n Internal High-Power"
- note added: "BTLE Variants (mutually exclusive)\n - External\n - Internal High-Power\n - Internal"
- note added: "Bluetooth Module"
- note added: "Bluetooth Programming Header"
- note added: "I2C Light Sensor"
- note added: "I2C Pull-ups"
- note added: "Programming Pull-ups"
- note added: "Programming Variant: Off-board"
- note added: "Programming Variant: On-board"
- note added: "Programming Variants (mutually exclusive)\n - On-board\n - Off-board"
- note added: "RJ45 Jack"
- note added: "RS422 Level Shifter"
- note added: "USB Power"
- note added: "User Interface"
- note added: "WiFi Activity LED"
- note added: "WiFi Module"
- note added: "WiFi Provisioning Button"
- note removed: "Auto-reset (programming)"
- note removed: "High-Power BTLE"
- note removed: "LED Indicators"
- note removed: "Power Control to External BTLE"
- note removed: "RS422 converter and RJ45 to External BTLE"
- note removed: "USB Power and Debug UART"
- note removed: "WiFi Module\nLow-Power BTLE"
- moved on the sheet: C1, C2, C3, C4, J2, Q3, R10, R14, R15, R16, R17, U1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
